Commit message: DPGG

File: Assets/AGV2.urdf (robot description, URDF)
Before this commit: robot macroed, 9 links, 8 joints
Links:
- link base_link: mass 0.5 -> 5
- link left_back_wheel: mass 0.3 -> 1
- link left_front_wheel: mass 0.3 -> 1
- link right_back_wheel: mass 0.3 -> 1
- link right_front_wheel: mass 0.3 -> 1
